File: Hardware/Production/Qwiic_Iridium_9603N-Panel.brd (EAGLE design)
At the start: 173.5 x 173.5 mm, 807 parts, among them J1 IRIDIUM_9603N, J10 PTH, J13 ISP, J14 U.FL, J15 IRIDIUM_9603N, J18 PTH, J21 ISP, J22 U.FL, J23 IRIDIUM_9603N, J26 PTH, J29 ISP, J3 PTH, J30 U.FL, J31 IRIDIUM_9603N, J34 PTH, J37 ISP, J38 U.FL, J39 IRIDIUM_9603N, J42 PTH, J45 ISP, J46 U.FL, J47 IRIDIUM_9603N, J50 PTH, J53 ISP, J54 U.FL, J55 IRIDIUM_9603N, J58 PTH, J6 ISP, J61 ISP, J62 U.FL, J63 IRIDIUM_9603N, J66 PTH, J69 ISP, J7 U.FL, J70 U.FL, J71 IRIDIUM_9603N, Q1 DMG3414U-7, Q2 DMG3414U-7, Q3 DMG3414U-7, Q4 DMG3414U-7, Q5 DMG3414U-7, Q6 DMG3414U-7, Q7 DMG3414U-7, Q8 DMG3414U-7, Q9 DMG3414U-7, U1 ATTINY841-ARDUINO, U10 ATTINY841-ARDUINO, U11 LTC3225EDDB#TRMPBF, U12 ADM4210-1, U13 ATTINY841-ARDUINO, U14 LTC3225EDDB#TRMPBF, U15 ADM4210-1, U16 ATTINY841-ARDUINO, U17 LTC3225EDDB#TRMPBF, U18 ADM4210-1, U19 ATTINY841-ARDUINO, U2 LTC3225EDDB#TRMPBF, U20 LTC3225EDDB#TRMPBF, U21 ADM4210-1, U22 ATTINY841-ARDUINO, U23 LTC3225EDDB#TRMPBF, U24 ADM4210-1, U25 ATTINY841-ARDUINO, U26 LTC3225EDDB#TRMPBF, U27 ADM4210-1, U3 ADM4210-1, U4 ATTINY841-ARDUINO, U5 LTC3225EDDB#TRMPBF, U6 ADM4210-1, U7 ATTINY841-ARDUINO, U8 LTC3225EDDB#TRMPBF, U9 ADM4210-1

Commit message: Adding x02 regular and production files.
Parts:
- JP10, JP11, JP12, JP18, JP19, JP21, JP22, JP28, JP29, JP3, JP31, JP32, JP38, JP39, JP4, JP41, JP42, JP48, JP49, JP51, JP52, JP58, JP59, JP61, JP62, JP68, JP69, JP71, JP72, JP78, JP79, JP81, JP82, JP88, JP89, JP9: device SparkFun:STAND-OFF -> SparkFun-Hardware:STAND-OFF
- JP13, JP14, JP15, JP16, JP23, JP24, JP25, JP26, JP33, JP34, JP35, JP36, JP43, JP44, JP45, JP46, JP5, JP53, JP54, JP55, JP56, JP6, JP63, JP64, JP65, JP66, JP7, JP73, JP74, JP75, JP76, JP8, JP83, JP84, JP85, JP86: value FIDUCIALUFIDUCIAL -> FIDUCIAL1X2; device SparkFun:MICRO-FIDUCIAL -> SparkFun-Aesthetics:FIDUCIAL-1X2
- Q1, Q2, Q3, Q4, Q5, Q6, Q7, Q8, Q9: value DMG3414U-7 -> 5.8A/30V/35mΩ; device DMG3414U-7:SOT96P240X100-3N -> SparkFun-DiscreteSemi:SOT23-3
- R1, R110, R113, R12, R124, R15, R26, R29, R40, R43, R54, R57, R68, R71, R82, R85, R96, R99: device SparkFun-Resistors:0603 -> Qwiic_Iridium_9603N:0603
- U1: value ATTINY841-ARDUINO -> ATTINY841SOIC; device Qwiic_Iridium_9603N:SO14 -> Qwiic_Iridium_9603N:ATTINY841
- U10, U13, U16, U19, U22, U25, U4, U7: value ATTINY841-ARDUINO -> LTC3225EDDB#TRMPBF; device Qwiic_Iridium_9603N:SO14 -> Qwiic_Iridium_9603N:DFN300X200-10L
- U11, U14, U17, U20, U23, U26, U5, U8: value LTC3225EDDB#TRMPBF -> ADM4210-1; device Qwiic_Iridium_9603N:DFN300X200-10L -> Qwiic_Iridium_9603N:TSOT6
- U12, U15, U18, U21, U24, U27, U6, U9: value ADM4210-1 -> ATTINY841SOIC; device ADM4210:TSOT6 -> Qwiic_Iridium_9603N:ATTINY841
- U3: device ADM4210:TSOT6 -> Qwiic_Iridium_9603N:TSOT6
- moved Q1 51.4 mm to (80.5, 35.6), turned to 270 degrees
- moved Q2 51.2 mm to (29.2, 35.6), turned to 270 degrees
- moved U12 20.4 mm to (24.1, 70.5)
- moved U21 20.4 mm to (24.1, 121.8)
- moved U15 20.4 mm to (75.4, 70.5)
- moved U18 20.4 mm to (126.7, 70.5)
- moved U24 20.4 mm to (75.4, 121.8)
- moved U27 20.4 mm to (126.7, 121.8)
- moved U6 20.4 mm to (75.4, 19.2)
- moved U9 20.4 mm to (126.7, 19.2)
- moved U25 12.5 mm to (133.2, 132.3)
- moved U7 12.5 mm to (133.2, 29.7)
- moved U19 12.5 mm to (30.6, 132.3)
- moved U22 12.5 mm to (81.9, 132.3)
- moved U16 12.5 mm to (133.2, 81.0)
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Connections:
- net !RST1: now also U6.4; no longer U4.4
- net !RST2: now also U9.4; no longer U7.4
- net !RST3: now also U12.4; no longer U10.4
- net !RST4: now also U15.4; no longer U13.4
- net !RST5: now also U18.4; no longer U16.4
- net !RST6: now also U21.4; no longer U19.4
- net !RST7: now also U24.4; no longer U22.4
- net !RST8: now also U27.4; no longer U25.4
- net !SHDN1: now also U4.4, U6.2; no longer U4.2, U5.4
- net !SHDN2: now also U7.4, U9.2; no longer U7.2, U8.4
- net !SHDN3: now also U10.4, U12.2; no longer U10.2, U11.4
- net !SHDN4: now also U13.4, U15.2; no longer U13.2, U14.4
- net !SHDN5: now also U16.4, U18.2; no longer U16.2, U17.4
- net !SHDN6: now also U19.4, U21.2; no longer U19.2, U20.4
- net !SHDN7: now also U22.4, U24.2; no longer U22.2, U23.4
- net !SHDN8: now also U25.4, U27.2; no longer U25.2, U26.4
- net 3.3V1: now also U4.6, U4.9, U6.1; no longer U4.1, U5.6, U5.9
- net 3.3V2: now also U7.6, U7.9, U9.1; no longer U7.1, U8.6, U8.9
- net 3.3V3: now also U10.6, U10.9, U12.1; no longer U10.1, U11.6, U11.9
- net 3.3V4: now also U13.6, U13.9, U15.1; no longer U13.1, U14.6, U14.9
- net 3.3V5: now also U16.6, U16.9, U18.1; no longer U16.1, U17.6, U17.9
- net 3.3V6: now also U19.6, U19.9, U21.1; no longer U19.1, U20.6, U20.9
- net 3.3V7: now also U22.6, U22.9, U24.1; no longer U22.1, U23.6, U23.9
- net 3.3V8: now also U25.6, U25.9, U27.1; no longer U25.1, U26.6, U26.9
- net EXT_PWR: now also Q2.2; no longer Q1.2
- net EXT_PWR1: now also Q1.2; no longer Q2.2
- net GND1: now also U4.11, U4.8, U5.2, U6.14; no longer U4.14, U5.11, U5.8, U6.2
- net GND2: now also U7.11, U7.8, U8.2, U9.14; no longer U7.14, U8.11, U8.8, U9.2
- net GND3: now also U10.11, U10.8, U11.2, U12.14; no longer U10.14, U11.11, U11.8, U12.2
- net GND4: now also U13.11, U13.8, U14.2, U15.14; no longer U13.14, U14.11, U14.8, U15.2
- net GND5: now also U16.11, U16.8, U17.2, U18.14; no longer U16.14, U17.11, U17.8, U18.2
- net GND6: now also U19.11, U19.8, U20.2, U21.14; no longer U19.14, U20.11, U20.8, U21.2
- net GND7: now also U22.11, U22.8, U23.2, U24.14; no longer U22.14, U23.11, U23.8, U24.2
- net GND8: now also U25.11, U25.8, U26.2, U27.14; no longer U25.14, U26.11, U26.8, U27.2
- net LTC3225_VOUT1: now also U4.10, U5.6; no longer U5.10, U6.6
- net LTC3225_VOUT2: now also U7.10, U8.6; no longer U8.10, U9.6
- net LTC3225_VOUT3: now also U10.10, U11.6; no longer U11.10, U12.6
- net LTC3225_VOUT4: now also U13.10, U14.6; no longer U14.10, U15.6
- net LTC3225_VOUT5: now also U16.10, U17.6; no longer U17.10, U18.6
- net LTC3225_VOUT6: now also U19.10, U20.6; no longer U20.10, U21.6
- net LTC3225_VOUT7: now also U22.10, U23.6; no longer U23.10, U24.6
- net LTC3225_VOUT8: now also U25.10, U26.6; no longer U26.10, U27.6
- net MISO1: now also U6.8; no longer U4.8
- net MISO2: now also U9.8; no longer U7.8
- net MISO3: now also U12.8; no longer U10.8
- net MISO4: now also U15.8; no longer U13.8
- net MISO5: now also U18.8; no longer U16.8
- net MISO6: now also U21.8; no longer U19.8
- net MISO7: now also U24.8; no longer U22.8
- net MISO8: now also U27.8; no longer U25.8
- net N$100: now also U19.7; no longer U20.7
- net N$101: now also U19.3; no longer U20.3
- net N$107: now also U20.5; no longer U21.5
- net N$109: now also U20.4; no longer U21.4
- net N$111: now also U20.1; no longer U21.1
- net N$114: now also U22.2; no longer U23.2
- net N$115: now also U22.1; no longer U23.1
- net N$116: now also U22.7; no longer U23.7
- net N$117: now also U22.3; no longer U23.3
- net N$12: now also Q2.1; no longer Q1.1
- net N$123: now also U23.5; no longer U24.5
- net N$125: now also U23.4; no longer U24.4
- net N$127: now also U23.1; no longer U24.1
- net N$130: now also U25.2; no longer U26.2
- net N$131: now also U25.1; no longer U26.1
- net N$132: now also U25.7; no longer U26.7
- net N$133: now also U25.3; no longer U26.3
- net N$139: now also U26.5; no longer U27.5
- net N$141: now also U26.4; no longer U27.4
- net N$143: now also U26.1; no longer U27.1
- net N$18: now also U4.2; no longer U5.2
- net N$19: now also U4.1; no longer U5.1
- net N$20: now also U4.7; no longer U5.7
- net N$21: now also U4.3; no longer U5.3
- net N$27: now also Q1.3, U5.5; no longer Q2.3, U6.5
- net N$28: now also Q1.1; no longer Q2.1
- net N$29: now also U5.4; no longer U6.4
- net N$31: now also U5.1; no longer U6.1
- net N$34: now also U7.2; no longer U8.2
- net N$35: now also U7.1; no longer U8.1
- net N$36: now also U7.7; no longer U8.7
- net N$37: now also U7.3; no longer U8.3
- net N$43: now also U8.5; no longer U9.5
- net N$45: now also U8.4; no longer U9.4
- net N$47: now also U8.1; no longer U9.1
- net N$50: now also U10.2; no longer U11.2
- net N$51: now also U10.1; no longer U11.1
- net N$52: now also U10.7; no longer U11.7
- net N$53: now also U10.3; no longer U11.3
- net N$59: now also U11.5; no longer U12.5
- net N$61: now also U11.4; no longer U12.4
- net N$63: now also U11.1; no longer U12.1
- net N$66: now also U13.2; no longer U14.2
- net N$67: now also U13.1; no longer U14.1
- net N$68: now also U13.7; no longer U14.7
- net N$69: now also U13.3; no longer U14.3
- net N$75: now also U14.5; no longer U15.5
- net N$77: now also U14.4; no longer U15.4
- net N$79: now also U14.1; no longer U15.1
- net N$8: now also Q2.3; no longer Q1.3
- net N$82: now also U16.2; no longer U17.2
- net N$83: now also U16.1; no longer U17.1
- net N$84: now also U16.7; no longer U17.7
- net N$85: now also U16.3; no longer U17.3
- net N$91: now also U17.5; no longer U18.5
- net N$93: now also U17.4; no longer U18.4
- net N$95: now also U17.1; no longer U18.1
- net N$98: now also U19.2; no longer U20.2
- net N$99: now also U19.1; no longer U20.1
- net NA1: now also U6.6; no longer U4.6
- net NA2: now also U9.6; no longer U7.6
- net NA3: now also U12.6; no longer U10.6
- net NA4: now also U15.6; no longer U13.6
- net NA5: now also U18.6; no longer U16.6
- net NA6: now also U21.6; no longer U19.6
- net NA7: now also U24.6; no longer U22.6
- net NA8: now also U27.6; no longer U25.6
- net ON_OFF1: now also U6.13; no longer U4.13
- net ON_OFF2: now also U9.13; no longer U7.13
- net ON_OFF3: now also U12.13; no longer U10.13
- net ON_OFF4: now also U15.13; no longer U13.13
- net ON_OFF5: now also U18.13; no longer U16.13
- net ON_OFF6: now also U21.13; no longer U19.13
- net ON_OFF7: now also U24.13; no longer U22.13
- net ON_OFF8: now also U27.13; no longer U25.13
- net PGOOD1: now also U6.5; no longer U5.5
- net PGOOD2: now also U9.5; no longer U8.5
- net PGOOD3: now also U12.5; no longer U11.5
- net PGOOD4: now also U15.5; no longer U14.5
- net PGOOD5: now also U18.5; no longer U17.5
- net PGOOD6: now also U21.5; no longer U20.5
- net PGOOD7: now also U24.5; no longer U23.5
- net PGOOD8: now also U27.5; no longer U26.5
- net PWR_EN1: now also U5.3, U6.10; no longer U4.10, U6.3
- net PWR_EN2: now also U8.3, U9.10; no longer U7.10, U9.3
- net PWR_EN3: now also U11.3, U12.10; no longer U10.10, U12.3
- net PWR_EN4: now also U14.3, U15.10; no longer U13.10, U15.3
- net PWR_EN5: now also U17.3, U18.10; no longer U16.10, U18.3
- net PWR_EN6: now also U20.3, U21.10; no longer U19.10, U21.3
- net PWR_EN7: now also U23.3, U24.10; no longer U22.10, U24.3
- net PWR_EN8: now also U26.3, U27.10; no longer U25.10, U27.3
- net RI1: now also U6.3; no longer U4.3
- net RI2: now also U9.3; no longer U7.3
- net RI3: now also U12.3; no longer U10.3
- net RI4: now also U15.3; no longer U13.3
- net RI5: now also U18.3; no longer U16.3
- net RI6: now also U21.3; no longer U19.3
- net RI7: now also U24.3; no longer U22.3
- net RI8: now also U27.3; no longer U25.3
- net RX(OUT)1: now also U6.11; no longer U4.11
- net RX(OUT)2: now also U9.11; no longer U7.11
- net RX(OUT)3: now also U12.11; no longer U10.11
- net RX(OUT)4: now also U15.11; no longer U13.11
- net RX(OUT)5: now also U18.11; no longer U16.11
- net RX(OUT)6: now also U21.11; no longer U19.11
- net RX(OUT)7: now also U24.11; no longer U22.11
- net RX(OUT)8: now also U27.11; no longer U25.11
- net SCL1: now also U6.9; no longer U4.9
- net SCL2: now also U9.9; no longer U7.9
- net SCL3: now also U12.9; no longer U10.9
- net SCL4: now also U15.9; no longer U13.9
- net SCL5: now also U18.9; no longer U16.9
- net SCL6: now also U21.9; no longer U19.9
- net SCL7: now also U24.9; no longer U22.9
- net SCL8: now also U27.9; no longer U25.9
- net SDA1: now also U6.7; no longer U4.7
- net SDA2: now also U9.7; no longer U7.7
- net SDA3: now also U12.7; no longer U10.7
- net SDA4: now also U15.7; no longer U13.7
- net SDA5: now also U18.7; no longer U16.7
- net SDA6: now also U21.7; no longer U19.7
- net SDA7: now also U24.7; no longer U22.7
- net SDA8: now also U27.7; no longer U25.7
- net TX(IN)1: now also U6.12; no longer U4.12
- net TX(IN)2: now also U9.12; no longer U7.12
- net TX(IN)3: now also U12.12; no longer U10.12
- net TX(IN)4: now also U15.12; no longer U13.12
- net TX(IN)5: now also U18.12; no longer U16.12
- net TX(IN)6: now also U21.12; no longer U19.12
- net TX(IN)7: now also U24.12; no longer U22.12
- net TX(IN)8: now also U27.12; no longer U25.12
Routing:
- net GND3: track 42.4 -> 43.0 mm, vias 44 -> 45
- net GND: track 42.4 -> 43.0 mm, vias 44 -> 45
- net GND5: track 42.4 -> 43.0 mm, vias 44 -> 45
- net GND4: track 42.4 -> 43.0 mm, vias 44 -> 45
- net GND2: track 42.4 -> 43.0 mm, vias 44 -> 45
- net GND1: track 42.4 -> 43.0 mm, vias 44 -> 45
- net GND6: track 42.4 -> 43.0 mm, vias 44 -> 45
- net GND8: track 42.4 -> 43.0 mm, vias 44 -> 45
- net GND7: track 42.4 -> 43.0 mm, vias 44 -> 45
- net PGOOD6: track 71.9 -> 72.4 mm
- net PGOOD4: track 71.9 -> 72.4 mm
- net PGOOD2: track 71.9 -> 72.4 mm
- net PGOOD1: track 71.9 -> 72.4 mm
- net PGOOD: track 71.9 -> 72.4 mm
- net PGOOD8: track 71.9 -> 72.4 mm
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Other:
- board text added: "X02"
- board text removed: "X0.1"
